File: wifi_ESP-01_opto_rele/ESP01.sch (KiCad schematic (older format))
At the start: 14 parts, among them J1 Conn_02x04_Odd_Even_MountingP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, J4 Conn_01x02, J5 Conn_01x02, Q3 BC547, Q4 BC547, U1 LD1117S33TR_SOT223

Commit message: Correcciones_revisor
Parts:
- renumbered C1 to C201, C2 to C202, J4 to J201, J5 to J202, J1 to J203, JP1 to JP201, JP2 to JP202, Q3 to Q201, Q4 to Q202, R5 to R201, R6 to R202, R7 to R203, R8 to R204, U1 to U201
Other:
- note added: "(3.3v)"
- note added: "ESP01: Módulo wifi (ver documentación anexa)"
- note added: "J201: Conector para voltaje de entrada 5v señal de control"
- note added: "J202: Conector para fuente externa"
- note added: "JP201: Conectar para trabajar con fuentes acopladas"
- note added: "JP202: Conectar para trabajar con tierras acopladas"
- moved on the sheet: J201, J202, JP201, JP202

Commit message: correcciones v2
Parts:
- J203: footprint Connector_PinSocket_2.54mm:PinSocket_2x04_P2.54mm_Vertical -> w_conn_mkds:PinSocket_2x04_P2.54mm_Vertical
Other:
- note added: "1 GND"
- note added: "2 GPIO2"
- note added: "3 GPIO0"
- note added: "4 RXD"
- note added: "CH_PD 6"
- note added: "RESET 7"
- note added: "TXD 5"
- note added: "VCC 8"
Changed lines of the file:
@@
 Comp "FIUBA-CESE"
 Comment1 "Autor: Christian Yánez"
-Comment2 "Copyright (c) 2018, CESE 6ta Co FIUBA"
-Comment3 ""
+Comment2 "Licencia: https://github.com/Christianyf/CESE_6Co_PCB/blob/master/licencia.txt"
+Comment3 "Copyright (c) 2018, CESE 6ta Co FIUBA"
 Comment4 ""
 $EndDescr
@@
 L power:GNDA #PWR0207
 U 1 1 5BBAEAD6
-P 6300 3050
-F 0 "#PWR0207" H 6300 2800 50  0001 C CNN
-F 1 "GNDA" H 6305 2877 50  0000 C CNN
-F 2 "" H 6300 3050 50  0001 C CNN
-F 3 "" H 6300 3050 50  0001 C CNN
-	1    6300 3050
+P 6300 3300
+F 0 "#PWR0207" H 6300 3050 50  0001 C CNN
+F 1 "GNDA" H 6305 3127 50  0000 C CNN
+F 2 "" H 6300 3300 50  0001 C CNN
+F 3 "" H 6300 3300 50  0001 C CNN
+	1    6300 3300
 	1    0    0    -1
 $EndComp
@@
 	7850 1950 7850 2150
 Wire Wire Line
-	6300 3050 6050 3050
-Wire Wire Line
 	6800 5000 7050 5000
 Wire Wire Line
@@
 F 0 "J203" H 5850 3000 50  0000 L CNN
 F 1 "Conn_02x04_Odd_Even_MountingPin" H 5250 2900 50  0000 L CNN
-F 2 "Connector_PinSocket_2.54mm:PinSocket_2x04_P2.54mm_Vertical" H 5850 3550 50  0001 C CNN
+F 2 "w_conn_mkds:PinSocket_2x04_P2.54mm_Vertical" H 5850 3550 50  0001 C CNN
 F 3 "~" H 5850 3550 50  0001 C CNN
 	1    5850 3550
@@
 Wire Wire Line
 	6800 3550 6800 2900
-Wire Wire Line
-	6050 3050 6050 3450
 Wire Wire Line
 	6050 3650 6800 3650
@@
 Text Notes 3350 3050 0    98   ~ 0
 Fuente regulada 3.3v
-Text Notes 5250 2700 0    98   ~ 0
+Text Notes 5250 2250 0    98   ~ 0
 Conector para\nmódulo ESP01\n    externo
 Text Notes 7400 1550 0    98   ~ 0
@@
 Wire Notes Line
 	4100 3400 4100 3100
-Wire Notes Line
-	5800 3300 5800 2800
 Text Notes 750  6450 0    50   ~ 0
 ESP01: Módulo wifi (ver documentación anexa)
@@
 Text Notes 750  7050 0    50   ~ 0
 J202: Conector para fuente externa
+Wire Notes Line
+	5700 3150 5700 2750
+Wire Notes Line
+	5700 2750 5900 2750
+Wire Notes Line
+	5900 2750 5900 3150
+Wire Notes Line
+	5700 3150 5900 3150
+Text Notes 5950 2800 0    50   ~ 0
+1 GND
+Text Notes 5950 2900 0    50   ~ 0
+2 GPIO2
+Text Notes 5950 3050 0    50   ~ 0
+3 GPIO0
+Text Notes 5950 3150 0    50   ~ 0
+4 RXD
+Text Notes 5450 2800 0    50   ~ 0
+TXD 5
+Text Notes 5350 2900 0    50   ~ 0
+CH_PD 6
+Text Notes 5350 3050 0    50   ~ 0
+RESET 7
+Text Notes 5450 3150 0    50   ~ 0
+VCC 8
+Wire Wire Line
+	6050 3450 6050 3250
+Wire Wire Line
+	6050 3250 6300 3250
+Wire Wire Line
+	6300 3250 6300 3300
+Wire Notes Line
+	5800 3350 5800 3200
+Wire Notes Line
+	5800 2650 5800 2350
 $EndSCHEMATC
