File: wifi_ESP-01_opto_rele/Opto-acople.sch (KiCad schematic (older format))
At the start: 16 parts, among them J2 Conn_01x03, J3 Conn_01x03, K1 G5LE-1, K2 G5LE-1, Q1 BC547, Q2 BC547, U2 PC817, U3 PC817

Commit message: Segunda revisión
Parts:
- added F1, F2, F3: MountingHole, Fiducial:Fiducial_1mm_Dia_2mm_Outer, symbol Mechanical:MountingHole
Changed lines of the file:
@@
 EESchema Schematic File Version 4
+LIBS:wifi_ESP-01_opto_rele-cache
 EELAYER 26 0
 EELAYER END
@@
 Text Label 7500 2350 2    50   ~ 0
 COM0
+$Comp
+L Mechanical:MountingHole F1
+U 1 1 5BBC1A9F
+P 4200 6150
+F 0 "F1" H 4300 6196 50  0000 L CNN
+F 1 "MountingHole" H 4300 6105 50  0000 L CNN
+F 2 "Fiducial:Fiducial_1mm_Dia_2mm_Outer" H 4200 6150 50  0001 C CNN
+F 3 "~" H 4200 6150 50  0001 C CNN
+	1    4200 6150
+	1    0    0    -1
+$EndComp
+$Comp
+L Mechanical:MountingHole F2
+U 1 1 5BBC1AED
+P 4200 6400
+F 0 "F2" H 4300 6446 50  0000 L CNN
+F 1 "MountingHole" H 4300 6355 50  0000 L CNN
+F 2 "Fiducial:Fiducial_1mm_Dia_2mm_Outer" H 4200 6400 50  0001 C CNN
+F 3 "~" H 4200 6400 50  0001 C CNN
+	1    4200 6400
+	1    0    0    -1
+$EndComp
+$Comp
+L Mechanical:MountingHole F3
+U 1 1 5BBC1B33
+P 5050 6150
+F 0 "F3" H 5150 6196 50  0000 L CNN
+F 1 "MountingHole" H 5150 6105 50  0000 L CNN
+F 2 "Fiducial:Fiducial_1mm_Dia_2mm_Outer" H 5050 6150 50  0001 C CNN
+F 3 "~" H 5050 6150 50  0001 C CNN
+	1    5050 6150
+	1    0    0    -1
+$EndComp
 $EndSCHEMATC

Commit message: Correcciones_revisor
Parts:
- renumbered D1 to D301, D2 to D302, D3 to D303, D4 to D304, F1 to F301, F2 to F302, F3 to F303, J2 to J301, J3 to J302, K1 to K301, K2 to K302, Q1 to Q301, Q2 to Q302, R1 to R301, R2 to R302, R3 to R303, R4 to R304, U2 to U301, U3 to U302
Changed lines of the file:
@@
 Comp "FIUBA-CESE"
 Comment1 "Autor: Christian Yánez"
-Comment2 ""
+Comment2 "Copyright (c) 2018, CESE 6ta Co FIUBA"
 Comment3 ""
 Comment4 ""
@@
 P 3500 2300
 AR Path="/5BBC390B" Ref="R?"  Part="1"
-AR Path="/5BBC31E0/5BBC390B" Ref="R1"  Part="1"
-F 0 "R1" H 3570 2346 50  0000 L CNN
+AR Path="/5BBC31E0/5BBC390B" Ref="R301"  Part="1"
+F 0 "R301" H 3570 2346 50  0000 L CNN
 F 1 "200" H 3570 2255 50  0000 L CNN
 F 2 "Resistor_SMD:R_0805_2012Metric_Pad1.15x1.40mm_HandSolder" V 3430 2300 50  0001 C CNN
@@
 P 3500 3300
 AR Path="/5BBC3912" Ref="D?"  Part="1"
-AR Path="/5BBC31E0/5BBC3912" Ref="D1"  Part="1"
-F 0 "D1" V 3538 3183 50  0000 R CNN
+AR Path="/5BBC31E0/5BBC3912" Ref="D301"  Part="1"
+F 0 "D301" V 3538 3183 50  0000 R CNN
 F 1 "LED" V 3447 3183 50  0000 R CNN
 F 2 "LED_SMD:LED_0805_2012Metric_Pad1.15x1.40mm_HandSolder" H 3500 3300 50  0001 C CNN
@@
 P 3800 2850
 AR Path="/5BBC3919" Ref="U?"  Part="1"
-AR Path="/5BBC31E0/5BBC3919" Ref="U2"  Part="1"
-F 0 "U2" H 3800 3175 50  0000 C CNN
+AR Path="/5BBC31E0/5BBC3919" Ref="U301"  Part="1"
+F 0 "U301" H 3800 3175 50  0000 C CNN
 F 1 "PC817" H 3800 3084 50  0000 C CNN
 F 2 "Package_DIP:DIP-4_W7.62mm" H 3600 2650 50  0001 L CIN
@@
 P 5400 2300
 AR Path="/5BBC3920" Ref="D?"  Part="1"
-AR Path="/5BBC31E0/5BBC3920" Ref="D3"  Part="1"
-F 0 "D3" V 5354 2379 50  0000 L CNN
+AR Path="/5BBC31E0/5BBC3920" Ref="D303"  Part="1"
+F 0 "D303" V 5354 2379 50  0000 L CNN
 F 1 "1N4148" V 5445 2379 50  0000 L CNN
 F 2 "Diode_SMD:D_0805_2012Metric_Pad1.15x1.40mm_HandSolder" H 5400 2125 50  0001 C CNN
@@
 P 6300 4550
 AR Path="/5BBC3927" Ref="K?"  Part="1"
-AR Path="/5BBC31E0/5BBC3927" Ref="K2"  Part="1"
-F 0 "K2" H 6730 4596 50  0000 L CNN
+AR Path="/5BBC31E0/5BBC3927" Ref="K302"  Part="1"
+F 0 "K302" H 6730 4596 50  0000 L CNN
 F 1 "G5LE-1" H 6730 4505 50  0000 L CNN
 F 2 "Relay_THT:Relay_SPDT_Omron-G5LE-1" H 6750 4500 50  0001 L CNN
@@
 P 5300 2950
 AR Path="/5BBC392E" Ref="Q?"  Part="1"
-AR Path="/5BBC31E0/5BBC392E" Ref="Q1"  Part="1"
-F 0 "Q1" H 5491 2996 50  0000 L CNN
+AR Path="/5BBC31E0/5BBC392E" Ref="Q301"  Part="1"
+F 0 "Q301" H 5491 2996 50  0000 L CNN
 F 1 "BC547" H 5491 2905 50  0000 L CNN
 F 2 "Package_TO_SOT_SMD:SOT-23" H 5500 2875 50  0001 L CIN
@@
 P 7800 2350
 AR Path="/5BBC3935" Ref="J?"  Part="1"
-AR Path="/5BBC31E0/5BBC3935" Ref="J2"  Part="1"
-F 0 "J2" H 7880 2392 50  0000 L CNN
+AR Path="/5BBC31E0/5BBC3935" Ref="J301"  Part="1"
+F 0 "J301" H 7880 2392 50  0000 L CNN
 F 1 "Conn_01x03" H 7880 2301 50  0000 L CNN
 F 2 "TerminalBlock:TerminalBlock_bornier-3_P5.08mm" H 7800 2350 50  0001 C CNN
@@
 P 7800 4550
 AR Path="/5BBC393C" Ref="J?"  Part="1"
-AR Path="/5BBC31E0/5BBC393C" Ref="J3"  Part="1"
-F 0 "J3" H 7880 4592 50  0000 L CNN
+AR Path="/5BBC31E0/5BBC393C" Ref="J302"  Part="1"
+F 0 "J302" H 7880 4592 50  0000 L CNN
 F 1 "Conn_01x03" H 7880 4501 50  0000 L CNN
 F 2 "TerminalBlock:TerminalBlock_bornier-3_P5.08mm" H 7800 4550 50  0001 C CNN
@@
 P 3500 4500
 AR Path="/5BBC3943" Ref="R?"  Part="1"
-AR Path="/5BBC31E0/5BBC3943" Ref="R2"  Part="1"
-F 0 "R2" H 3570 4546 50  0000 L CNN
+AR Path="/5BBC31E0/5BBC3943" Ref="R302"  Part="1"
+F 0 "R302" H 3570 4546 50  0000 L CNN
 F 1 "200" H 3570 4455 50  0000 L CNN
 F 2 "Resistor_SMD:R_0805_2012Metric_Pad1.15x1.40mm_HandSolder" V 3430 4500 50  0001 C CNN
@@
 P 3800 5050
 AR Path="/5BBC394A" Ref="U?"  Part="1"
-AR Path="/5BBC31E0/5BBC394A" Ref="U3"  Part="1"
-F 0 "U3" H 3800 5375 50  0000 C CNN
+AR Path="/5BBC31E0/5BBC394A" Ref="U302"  Part="1"
+F 0 "U302" H 3800 5375 50  0000 C CNN
 F 1 "PC817" H 3800 5284 50  0000 C CNN
 F 2 "Package_DIP:DIP-4_W7.62mm" H 3600 4850 50  0001 L CIN
@@
 P 3500 5500
 AR Path="/5BBC3951" Ref="D?"  Part="1"
-AR Path="/5BBC31E0/5BBC3951" Ref="D2"  Part="1"
-F 0 "D2" V 3538 5383 50  0000 R CNN
+AR Path="/5BBC31E0/5BBC3951" Ref="D302"  Part="1"
+F 0 "D302" V 3538 5383 50  0000 R CNN
 F 1 "LED" V 3447 5383 50  0000 R CNN
 F 2 "LED_SMD:LED_0805_2012Metric_Pad1.15x1.40mm_HandSolder" H 3500 5500 50  0001 C CNN
@@
 P 4550 2950
 AR Path="/5BBC3958" Ref="R?"  Part="1"
-AR Path="/5BBC31E0/5BBC3958" Ref="R3"  Part="1"
-F 0 "R3" V 4343 2950 50  0000 C CNN
+AR Path="/5BBC31E0/5BBC3958" Ref="R303"  Part="1"
+F 0 "R303" V 4343 2950 50  0000 C CNN
 F 1 "1k" V 4434 2950 50  0000 C CNN
 F 2 "Resistor_SMD:R_0805_2012Metric_Pad1.15x1.40mm_HandSolder" V 4480 2950 50  0001 C CNN
@@
 P 4550 5150
 AR Path="/5BBC395F" Ref="R?"  Part="1"
-AR Path="/5BBC31E0/5BBC395F" Ref="R4"  Part="1"
-F 0 "R4" V 4343 5150 50  0000 C CNN
+AR Path="/5BBC31E0/5BBC395F" Ref="R304"  Part="1"
+F 0 "R304" V 4343 5150 50  0000 C CNN
 F 1 "1k" V 4434 5150 50  0000 C CNN
 F 2 "Resistor_SMD:R_0805_2012Metric_Pad1.15x1.40mm_HandSolder" V 4480 5150 50  0001 C CNN
@@
 P 5300 5150
 AR Path="/5BBC3966" Ref="Q?"  Part="1"
-AR Path="/5BBC31E0/5BBC3966" Ref="Q2"  Part="1"
-F 0 "Q2" H 5491 5196 50  0000 L CNN
+AR Path="/5BBC31E0/5BBC3966" Ref="Q302"  Part="1"
+F 0 "Q302" H 5491 5196 50  0000 L CNN
 F 1 "BC547" H 5491 5105 50  0000 L CNN
 F 2 "Package_TO_SOT_SMD:SOT-23" H 5500 5075 50  0001 L CIN
@@
 P 5400 4500
 AR Path="/5BBC396D" Ref="D?"  Part="1"
-AR Path="/5BBC31E0/5BBC396D" Ref="D4"  Part="1"
-F 0 "D4" V 5354 4579 50  0000 L CNN
+AR Path="/5BBC31E0/5BBC396D" Ref="D304"  Part="1"
+F 0 "D304" V 5354 4579 50  0000 L CNN
 F 1 "1N4148" V 5445 4579 50  0000 L CNN
 F 2 "Diode_SMD:D_0805_2012Metric_Pad1.15x1.40mm_HandSolder" H 5400 4325 50  0001 C CNN
@@
 P 6300 2350
 AR Path="/5BBC3974" Ref="K?"  Part="1"
-AR Path="/5BBC31E0/5BBC3974" Ref="K1"  Part="1"
-F 0 "K1" H 6730 2396 50  0000 L CNN
+AR Path="/5BBC31E0/5BBC3974" Ref="K301"  Part="1"
+F 0 "K301" H 6730 2396 50  0000 L CNN
 F 1 "G5LE-1" H 6730 2305 50  0000 L CNN
 F 2 "Relay_THT:Relay_SPDT_Omron-G5LE-1" H 6750 2300 50  0001 L CNN
@@
 P 5400 3350
 AR Path="/5BBC397D" Ref="#PWR?"  Part="1"
-AR Path="/5BBC31E0/5BBC397D" Ref="#PWR0101"  Part="1"
-F 0 "#PWR0101" H 5400 3100 50  0001 C CNN
+AR Path="/5BBC31E0/5BBC397D" Ref="#PWR0304"  Part="1"
+F 0 "#PWR0304" H 5400 3100 50  0001 C CNN
 F 1 "GND" H 5405 3177 50  0000 C CNN
 F 2 "" H 5400 3350 50  0001 C CNN
@@
 P 3500 1800
 AR Path="/5BBC3986" Ref="#PWR?"  Part="1"
-AR Path="/5BBC31E0/5BBC3986" Ref="#PWR0102"  Part="1"
-F 0 "#PWR0102" H 3500 1650 50  0001 C CNN
+AR Path="/5BBC31E0/5BBC3986" Ref="#PWR0301"  Part="1"
+F 0 "#PWR0301" H 3500 1650 50  0001 C CNN
 F 1 "+5VA" H 3515 1973 50  0000 C CNN
 F 2 "" H 3500 1800 50  0001 C CNN
@@
 P 5400 1800
 AR Path="/5BBC39A1" Ref="#PWR?"  Part="1"
-AR Path="/5BBC31E0/5BBC39A1" Ref="#PWR0103"  Part="1"
-F 0 "#PWR0103" H 5400 1650 50  0001 C CNN
+AR Path="/5BBC31E0/5BBC39A1" Ref="#PWR0303"  Part="1"
+F 0 "#PWR0303" H 5400 1650 50  0001 C CNN
 F 1 "+5V" H 5415 1973 50  0000 C CNN
 F 2 "" H 5400 1800 50  0001 C CNN
@@
 P 3500 4000
 AR Path="/5BBC39AA" Ref="#PWR?"  Part="1"
-AR Path="/5BBC31E0/5BBC39AA" Ref="#PWR0104"  Part="1"
-F 0 "#PWR0104" H 3500 3850 50  0001 C CNN
+AR Path="/5BBC31E0/5BBC39AA" Ref="#PWR0302"  Part="1"
+F 0 "#PWR0302" H 3500 3850 50  0001 C CNN
 F 1 "+5VA" H 3515 4173 50  0000 C CNN
 F 2 "" H 3500 4000 50  0001 C CNN
@@
 P 5400 4000
 AR Path="/5BBC39BF" Ref="#PWR?"  Part="1"
-AR Path="/5BBC31E0/5BBC39BF" Ref="#PWR0105"  Part="1"
-F 0 "#PWR0105" H 5400 3850 50  0001 C CNN
+AR Path="/5BBC31E0/5BBC39BF" Ref="#PWR0305"  Part="1"
+F 0 "#PWR0305" H 5400 3850 50  0001 C CNN
 F 1 "+5V" H 5415 4173 50  0000 C CNN
 F 2 "" H 5400 4000 50  0001 C CNN
@@
 P 5400 5550
 AR Path="/5BBC39D2" Ref="#PWR?"  Part="1"
-AR Path="/5BBC31E0/5BBC39D2" Ref="#PWR0106"  Part="1"
-F 0 "#PWR0106" H 5400 5300 50  0001 C CNN
+AR Path="/5BBC31E0/5BBC39D2" Ref="#PWR0306"  Part="1"
+F 0 "#PWR0306" H 5400 5300 50  0001 C CNN
 F 1 "GND" H 5405 5377 50  0000 C CNN
 F 2 "" H 5400 5550 50  0001 C CNN
@@
 COM0
 $Comp
-L Mechanical:MountingHole F1
+L Mechanical:MountingHole F301
 U 1 1 5BBC1A9F
 P 4200 6150
-F 0 "F1" H 4300 6196 50  0000 L CNN
+F 0 "F301" H 4300 6196 50  0000 L CNN
 F 1 "MountingHole" H 4300 6105 50  0000 L CNN
 F 2 "Fiducial:Fiducial_1mm_Dia_2mm_Outer" H 4200 6150 50  0001 C CNN
@@
 $EndComp
 $Comp
-L Mechanical:MountingHole F2
+L Mechanical:MountingHole F302
 U 1 1 5BBC1AED
 P 4200 6400
-F 0 "F2" H 4300 6446 50  0000 L CNN
+F 0 "F302" H 4300 6446 50  0000 L CNN
 F 1 "MountingHole" H 4300 6355 50  0000 L CNN
 F 2 "Fiducial:Fiducial_1mm_Dia_2mm_Outer" H 4200 6400 50  0001 C CNN
@@
 $EndComp
 $Comp
-L Mechanical:MountingHole F3
+L Mechanical:MountingHole F303
 U 1 1 5BBC1B33
 P 5050 6150
-F 0 "F3" H 5150 6196 50  0000 L CNN
+F 0 "F303" H 5150 6196 50  0000 L CNN
 F 1 "MountingHole" H 5150 6105 50  0000 L CNN
 F 2 "Fiducial:Fiducial_1mm_Dia_2mm_Outer" H 5050 6150 50  0001 C CNN

Commit message: correcciones v2
Parts:
- removed F301, F302, F303: MountingHole, Fiducial:Fiducial_1mm_Dia_2mm_Outer, symbol Mechanical:MountingHole
Changed lines of the file:
@@
 Comp "FIUBA-CESE"
 Comment1 "Autor: Christian Yánez"
-Comment2 "Copyright (c) 2018, CESE 6ta Co FIUBA"
-Comment3 ""
+Comment2 "Licencia: https://github.com/Christianyf/CESE_6Co_PCB/blob/master/licencia.txt"
+Comment3 "Copyright (c) 2018, CESE 6ta Co FIUBA"
 Comment4 ""
 $EndDescr
@@
 Text Label 7500 2350 2    50   ~ 0
 COM0
-$Comp
-L Mechanical:MountingHole F301
-U 1 1 5BBC1A9F
-P 4200 6150
-F 0 "F301" H 4300 6196 50  0000 L CNN
-F 1 "MountingHole" H 4300 6105 50  0000 L CNN
-F 2 "Fiducial:Fiducial_1mm_Dia_2mm_Outer" H 4200 6150 50  0001 C CNN
-F 3 "~" H 4200 6150 50  0001 C CNN
-	1    4200 6150
-	1    0    0    -1
-$EndComp
-$Comp
-L Mechanical:MountingHole F302
-U 1 1 5BBC1AED
-P 4200 6400
-F 0 "F302" H 4300 6446 50  0000 L CNN
-F 1 "MountingHole" H 4300 6355 50  0000 L CNN
-F 2 "Fiducial:Fiducial_1mm_Dia_2mm_Outer" H 4200 6400 50  0001 C CNN
-F 3 "~" H 4200 6400 50  0001 C CNN
-	1    4200 6400
-	1    0    0    -1
-$EndComp
-$Comp
-L Mechanical:MountingHole F303
-U 1 1 5BBC1B33
-P 5050 6150
-F 0 "F303" H 5150 6196 50  0000 L CNN
-F 1 "MountingHole" H 5150 6105 50  0000 L CNN
-F 2 "Fiducial:Fiducial_1mm_Dia_2mm_Outer" H 5050 6150 50  0001 C CNN
-F 3 "~" H 5050 6150 50  0001 C CNN
-	1    5050 6150
-	1    0    0    -1
-$EndComp
 $EndSCHEMATC
