File: wifi_ESP-01_opto_rele/wifi_ESP-01_opto_rele.kicad_pcb (KiCad board)
At the start: 2 copper layers, 82.5 x 37.5 mm, 30 parts, among them J1 Conn_02x04_Odd_Even_MountingP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, J2 Conn_01x03, J3 Conn_01x03, J4 Conn_01x02, J5 Conn_01x02, K1 G5LE-1, K2 G5LE-1, Q1 BC547, Q2 BC547, Q3 BC547, Q4 BC547, U1 LD1117S33TR_SOT223, U2 PC817, U3 PC817

Commit message: Segunda revisión
Parts:
- added F1: MountingHole, Fiducial:Fiducial_1mm_Dia_2mm_Outer, F.Cu at (112.0, 92.2)
- added F2: MountingHole, Fiducial:Fiducial_1mm_Dia_2mm_Outer, F.Cu at (85.5, 72.2)
- added F3: MountingHole, Fiducial:Fiducial_1mm_Dia_2mm_Outer, F.Cu at (121.8, 59.8)
Routing:
- net Net-(Q4-Pad2): track 3.18 -> 2.53 mm
Other:
- rule pad_to_mask_clearance: 0.2 -> 0
- board text added: "ESP01-OPTO V1.0"
- board text added: "Grilla: 0,25mm Pista:0,8mm Margen global:0,8mm Vía:1,5mm Drill:0,8mm Terminación superficial: ninguna Fabricación nacional"
- board text added: "IND. ARG"

Commit message: correcciones pcb
Parts:
- removed D4: 1N4148, Diode_SMD:D_0805_2012Metric_Pad1.15x1.40mm_HandSolder
- removed R4: 1k, Resistor_SMD:R_0805_2012Metric_Pad1.15x1.40mm_HandSolder
- added D304: 1N4148, Diode_SMD:D_0805_2012Metric_Pad1.15x1.40mm_HandSolder, F.Cu at (118.2, 77.8)
- added R304: 1k, Resistor_SMD:R_0805_2012Metric_Pad1.15x1.40mm_HandSolder, F.Cu at (118.2, 81.0)
- renumbered C1 to C201, C2 to C202, D1 to D301, D2 to D302, D3 to D303, F1 to F301, F2 to F302, F3 to F303, J4 to J201, J5 to J202, J1 to J203, J2 to J301, J3 to J302, JP1 to JP201, JP2 to JP202, K1 to K301, K2 to K302, Q3 to Q201, Q4 to Q202, Q1 to Q301, Q2 to Q302, R5 to R201, R6 to R202, R7 to R203, R8 to R204, R1 to R301, R2 to R302, R3 to R303, U1 to U201, U2 to U301, U3 to U302
Routing:
- net GNDA: track 93.4 -> 59.1 mm, vias 6 -> 7
- net GND: track 66.7 -> 62.2 mm
Other:
- net class Default: clearance 0.8 -> 0.6
- rule trace_clearance: 0.8 -> 0.6
- board text added: "1 Oz"
- board text added: "2X7628AT05"
- board text added: "4x7628M"
- board text added: "Grilla: 0,25mm Pista:0,6-0,8-1mm Margen global:0,8mm Vía:0,8mm Drill:0,4mm Terminación superficial: HASL Fabricación nacional"
- board text added: "L1 (Top)"
- board text added: "L2 (Bottom)"
- board text added: "Laminate Isola"
- board text added: "Prepeg Isola"
- board text added: "STACK-UP"
- board text removed: "Grilla: 0,25mm Pista:0,8mm Margen global:0,8mm Vía:1,5mm Drill:0,8mm Terminación superficial: ninguna Fabricación nacional"

Commit message: correcciones v2
Parts:
- removed F301, F302, F303: MountingHole, Fiducial:Fiducial_1mm_Dia_2mm_Outer
- added F101: MountingHole, Fiducial:Fiducial_1mm_Dia_2mm_Outer, F.Cu at (105.0, 88.2)
- added F102: MountingHole, Fiducial:Fiducial_1mm_Dia_2mm_Outer, F.Cu at (115.8, 59.5)
- added F103: MountingHole, Fiducial:Fiducial_1mm_Dia_2mm_Outer, F.Cu at (85.5, 72.0)
- J203: footprint Connector_PinSocket_2.54mm:PinSocket_2x04_P2.54mm_Vertical -> w_conn_mkds:PinSocket_2x04_P2.54mm_Vertical
- moved J301 25.0 mm to (141.0, 89.5)
- moved J302 25.0 mm to (159.2, 89.5)
- moved K301 10.0 mm to (135.8, 63.2)
- moved K302 10.0 mm to (154.0, 63.2)
- moved JP201 8.06 mm to (124.0, 65.2)
- moved JP202 3.64 mm to (124.0, 61.2)
- moved J201 1.50 mm to (88.0, 89.2)
Routing:
- net +5V: track 159.9 -> 105.8 mm
- net GND: track 62.2 -> 15.9 mm
- net /Opto-aclope/COM1: track 8.78 -> 26.3 mm
- net /Opto-aclope/COM0: track 8.78 -> 26.3 mm
- net Net-(J302-Pad3): track 24.5 -> 12.5 mm
- net Net-(J301-Pad1): track 24.3 -> 12.4 mm
- net Net-(J302-Pad1): track 24.3 -> 12.4 mm
- net Net-(J301-Pad3): track 24.4 -> 12.5 mm
- net GNDA: track 59.1 -> 49.0 mm, vias 7 -> 6
- net Net-(D304-Pad2): track 31.2 -> 36.4 mm
- net +5VA: track 113.5 -> 108.7 mm
- net Net-(C202-Pad1): track 27.6 -> 31.0 mm
- net /ESP01/GPIO0: track 23.3 -> 21.2 mm
- net Net-(D303-Pad2): track 13.4 -> 12.8 mm
Other:
- board text added: "Grilla: 0,25mm Pista:0,6-0,8mm Margen global:0,6mm Vía:0,8mm Drill:0,4mm Terminación superficial: HASL Fabricación nacional"
- board text removed: "Grilla: 0,25mm Pista:0,6-0,8-1mm Margen global:0,8mm Vía:0,8mm Drill:0,4mm Terminación superficial: HASL Fabricación nacional"
