File: wifi_ESP-01_opto_rele/wifi_ESP-01_opto_rele.sch (KiCad schematic (older format))
At the start: 0 parts

Commit message: correcciones v2
Parts:
- added F101, F102, F103: MountingHole, Fiducial:Fiducial_1mm_Dia_2mm_Outer, symbol Mechanical:MountingHole
Changed lines of the file:
@@
 Comp "FIUBA-CESE"
 Comment1 "Autor: Christian Yánez"
-Comment2 "Copyright (c) 2018, CESE 6ta Co FIUBA"
-Comment3 ""
+Comment2 "Licencia: https://github.com/Christianyf/CESE_6Co_PCB/blob/master/licencia.txt"
+Comment3 "Copyright (c) 2018, CESE 6ta Co FIUBA"
 Comment4 ""
 $EndDescr
@@
 Wire Wire Line
 	4900 3850 6700 3850
+$Comp
+L Mechanical:MountingHole F?
+U 1 1 5BF4B9C4
+P 5150 6500
+AR Path="/5BBC31E0/5BF4B9C4" Ref="F?"  Part="1"
+AR Path="/5BF4B9C4" Ref="F101"  Part="1"
+F 0 "F101" H 5250 6546 50  0000 L CNN
+F 1 "MountingHole" H 5250 6455 50  0000 L CNN
+F 2 "Fiducial:Fiducial_1mm_Dia_2mm_Outer" H 5150 6500 50  0001 C CNN
+F 3 "~" H 5150 6500 50  0001 C CNN
+	1    5150 6500
+	1    0    0    -1
+$EndComp
+$Comp
+L Mechanical:MountingHole F?
+U 1 1 5BF4B9CB
+P 5150 6750
+AR Path="/5BBC31E0/5BF4B9CB" Ref="F?"  Part="1"
+AR Path="/5BF4B9CB" Ref="F102"  Part="1"
+F 0 "F102" H 5250 6796 50  0000 L CNN
+F 1 "MountingHole" H 5250 6705 50  0000 L CNN
+F 2 "Fiducial:Fiducial_1mm_Dia_2mm_Outer" H 5150 6750 50  0001 C CNN
+F 3 "~" H 5150 6750 50  0001 C CNN
+	1    5150 6750
+	1    0    0    -1
+$EndComp
+$Comp
+L Mechanical:MountingHole F?
+U 1 1 5BF4B9D2
+P 6000 6500
+AR Path="/5BBC31E0/5BF4B9D2" Ref="F?"  Part="1"
+AR Path="/5BF4B9D2" Ref="F103"  Part="1"
+F 0 "F103" H 6100 6546 50  0000 L CNN
+F 1 "MountingHole" H 6100 6455 50  0000 L CNN
+F 2 "Fiducial:Fiducial_1mm_Dia_2mm_Outer" H 6000 6500 50  0001 C CNN
+F 3 "~" H 6000 6500 50  0001 C CNN
+	1    6000 6500
+	1    0    0    -1
+$EndComp
 $EndSCHEMATC
